File: SMU V1/main_io.kicad_sch (KiCad schematic)
At the start: 0 parts

Commit message: i forget what i changed
Parts:
- added C401, C402, C403, C404: 22u, Capacitor_SMD:C_0805_2012Metric_Pad1.18x1.45mm_HandSolder, symbol bfr_capacitors:CL21A226MAQNNNE
- added J401, J402: Connector, symbol bfr_connectors:DAQ_Connector
Connections:
- new net CANH: J401.4, J402.4
- new net CANL: J401.3, J402.3
- new net GND: C401.2, C402.2, C403.2, C404.2, J401.2, J402.2
- new net VBATT+: C401.1, C402.1, C403.1, C404.1, J401.1, J402.1

Commit message: halfway done with routing, still needs antenna
Parts:
- J401: footprint (none) -> Connector_Molex:Molex_Micro-Fit_3.0_43650-0400_1x04_P3.00mm_Horizontal; Alternate 1 https://www.digikey.ca/en/products/detail/molex/0436500401/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 -> Datasheet https://www.te.com/commerce/DocumentDelivery/DDEC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; Alternate 2 (none) -> https://www.digikey.com/en/products/detail/te-connectivity-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; Digikey P/N 17-2339204-4CT-ND -> WM1867-ND; Manufacturer TE Connectivity -> Molex; Manufacturer P/N 2339204-4 -> 0436500401; Mouser P/N 571-2339204-4 -> 538-43650-0401
- J402: footprint (none) -> Connector_Molex:Molex_Micro-Fit_3.0_43650-0400_1x04_P3.00mm_Horizontal; Alternate 1 https://www.digikey.ca/en/products/detail/molex/0436500401/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 -> Datasheet https://www.te.com/commerce/DocumentDelivery/DDEC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; Digikey P/N 17-2339204-4CT-ND -> WM1867-ND; Manufacturer TE Connectivity -> Molex; Manufacturer P/N 2339204-4 -> 0436500401; Mouser P/N 571-2339204-4 -> 538-43650-0401
Connections:
- net CANH renamed CAN+
- net CANL renamed CAN-
