File: SMU V1/gps.kicad_sch (KiCad schematic)
At the start: 1 part

Commit message: i forget what i changed
Parts:
- added C501: 33p, Capacitor_SMD:C_0402_1005Metric_Pad0.74x0.62mm_HandSolder, symbol bfr_capacitors:0402CG330J500NT
- added C502: 100n, Capacitor_SMD:C_0402_1005Metric_Pad0.74x0.62mm_HandSolder, symbol bfr_capacitors:CL05B104KO5NNNC
- added C503: 4.7u, Capacitor_SMD:C_0603_1608Metric_Pad1.08x0.95mm_HandSolder, symbol bfr_capacitors:CL10A475KO8NNNC
Connections:
- net PP3300_GPS_VBCKUP is gone; now on net PP3300_GPS_VCC: GPS501.22 (V_BCKUP)
- net GND: now also C501.2, C502.2, C503.2
- net PP3300_GPS_VCC: now also C501.1, C502.1, C503.1
- net GPS_UART_RX renamed GPS_UART.RX
- net GPS_UART_TX renamed GPS_UART.TX
Other:
- sheet GPS Power renamed GPS LDO
- sheet GPS LDO: file gps_power.kicad_sch -> low_noise_ldo.kicad_sch
- sheet GPS LDO ports: added LDO_EN, PP3300_VOUT, PP5000_VIN; removed PP3300_GPS_VCC, PP5000_VSUPP

Commit message: halfway done with routing, still needs antenna
Parts:
- added TP501: GPS_UART_RX, bfr_utilities:TestPoint_Keystone_5019_Miniature, symbol bfr_utilities:SMD_Test_Point
- added TP502: GPS_UART_TX, bfr_utilities:TestPoint_Keystone_5019_Miniature, symbol bfr_utilities:SMD_Test_Point
- added TP503: GPS_WKUP, bfr_utilities:TestPoint_Keystone_5019_Miniature, symbol bfr_utilities:SMD_Test_Point
- added TP504: GPS_1PPS, bfr_utilities:TestPoint_Keystone_5019_Miniature, symbol bfr_utilities:SMD_Test_Point
- added TP505: GPS_nRST, bfr_utilities:TestPoint_Keystone_5019_Miniature, symbol bfr_utilities:SMD_Test_Point
- added TP506: GPS_+3V3, bfr_utilities:TestPoint_Keystone_5019_Miniature, symbol bfr_utilities:SMD_Test_Point
- GPS501: footprint (none) -> bfr_sensors:Quectel LC49
Connections:
- net GPS_1PPS: now also TP504.1
- net GPS_UART.RX: now also TP501.1
- net GPS_UART.TX: now also TP502.1
- net GPS_WKUP: now also TP503.1
- net GPS_nRST: now also TP505.1
- net PP3300_GPS_VCC: now also TP506.1

Commit message: finished, should prob double check the high frequency stuff
Connections:
- net GPS_ANTENNA renamed GPS_ANTENNA_RF
- net GPS_MODE_OUTPUT renamed GPS_ANT_ON
- net GPS_VDD_RF renamed GPS_RF_VDD
Changed lines of the file:
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@@
 		)
 	)
-	(label "GPS_VDD_RF"
+	(label "GPS_RF_VDD"
 		(at 129.54 133.35 0)
 		(effects
@@
 		)
 	)
-	(label "GPS_ANTENNA"
+	(label "GPS_ANTENNA_RF"
 		(at 129.54 125.73 0)
 		(effects
@@
 		)
 	)
-	(hierarchical_label "GPS_VDD_RF"
+	(hierarchical_label "GPS_RF_VDD"
 		(shape output)
 		(at 156.21 133.35 0)
@@
 			)
 			(justify left)
-		)
-	)
-	(hierarchical_label "GPS_MODE_OUTPUT"
-		(shape output)
-		(at 64.77 125.73 180)
-		(effects
-			(font
-				(size 1.27 1.27)
-			)
-			(justify right)
 		)
 	)
@@
 		)
 	)
-	(hierarchical_label "GPS_ANTENNA"
+	(hierarchical_label "GPS_ANTENNA_RF"
 		(shape output)
 		(at 156.21 125.73 0)
