File: SMU V2/5V_buck.kicad_sch (KiCad schematic)
At the start: 15 parts, among them U901 TPS5430DDAR, U902 ETQ-P3M150KVN

Commit message: v2 layout
Parts:
- renumbered C901 to C1001, C902 to C1002, C903 to C1003, C904 to C1004, C905 to C1005, C906 to C1006, C907 to C1007, C908 to C1008, C909 to C1009, D901 to D1001, R901 to R1001, R902 to R1002, R903 to R1003, U901 to U1001, U902 to U1002
Changed lines of the file:
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@@
 		(dnp no)
 		(fields_autoplaced yes)
-		(property "Reference" "U902"
+		(property "Reference" "U1002"
 			(at 153.67 76.8349 90)
 			(effects
@@
 			(project "SMU V1"
 				(path "/1f58b889-96e6-4877-90a3-5a655db5910b/b9f10619-4e5b-45af-b866-c6815d605ed5/af802241-6422-4666-a084-41c36db8cc4c"
-					(reference "U902")
+					(reference "U1002")
 					(unit 1)
 				)
@@
 		(dnp no)
 		(fields_autoplaced yes)
-		(property "Reference" "C904"
+		(property "Reference" "C1004"
 			(at 113.03 74.93 90)
 			(effects
@@
 			(project "SMU V1"
 				(path "/1f58b889-96e6-4877-90a3-5a655db5910b/b9f10619-4e5b-45af-b866-c6815d605ed5/af802241-6422-4666-a084-41c36db8cc4c"
-					(reference "C904")
+					(reference "C1004")
 					(unit 1)
 				)
@@
 		(dnp no)
 		(fields_autoplaced yes)
-		(property "Reference" "#PWR0902"
+		(property "Reference" "#PWR01002"
 			(at 229.87 115.57 0)
 			(effects
@@
 			(project "SMU V1"
 				(path "/1f58b889-96e6-4877-90a3-5a655db5910b/b9f10619-4e5b-45af-b866-c6815d605ed5/af802241-6422-4666-a084-41c36db8cc4c"
-					(reference "#PWR0902")
+					(reference "#PWR01002")
 					(unit 1)
 				)
@@
 		(dnp no)
 		(fields_autoplaced yes)
-		(property "Reference" "C903"
+		(property "Reference" "C1003"
 			(at 83.82 59.69 90)
 			(effects
@@
 			(project ""
 				(path "/1f58b889-96e6-4877-90a3-5a655db5910b/b9f10619-4e5b-45af-b866-c6815d605ed5/af802241-6422-4666-a084-41c36db8cc4c"
-					(reference "C903")
+					(reference "C1003")
 					(unit 1)
 				)
@@
 		(dnp no)
 		(fields_autoplaced yes)
-		(property "Reference" "C909"
+		(property "Reference" "C1009"
 			(at 220.98 87.6299 0)
 			(effects
@@
 			(project "SMU V1"
 				(path "/1f58b889-96e6-4877-90a3-5a655db5910b/b9f10619-4e5b-45af-b866-c6815d605ed5/af802241-6422-4666-a084-41c36db8cc4c"
-					(reference "C909")
+					(reference "C1009")
 					(unit 1)
 				)
@@
 		(dnp no)
 		(fields_autoplaced yes)
-		(property "Reference" "D901"
+		(property "Reference" "D1001"
 			(at 138.43 89.8524 90)
 			(effects
@@
 			(project "SMU V1"
 				(path "/1f58b889-96e6-4877-90a3-5a655db5910b/b9f10619-4e5b-45af-b866-c6815d605ed5/af802241-6422-4666-a084-41c36db8cc4c"
-					(reference "D901")
+					(reference "D1001")
 					(unit 1)
 				)
@@
 		(dnp no)
 		(fields_autoplaced yes)
-		(property "Reference" "R902"
+		(property "Reference" "R1002"
 			(at 232.41 85.0899 90)
 			(effects
@@
 			(project "SMU V1"
 				(path "/1f58b889-96e6-4877-90a3-5a655db5910b/b9f10619-4e5b-45af-b866-c6815d605ed5/af802241-6422-4666-a084-41c36db8cc4c"
-					(reference "R902")
+					(reference "R1002")
 					(unit 1)
 				)
@@
 		(dnp no)
 		(fields_autoplaced yes)
-		(property "Reference" "U901"
+		(property "Reference" "U1001"
 			(at 93.98 74.93 0)
 			(effects
@@
 			(project "SMU V1"
 				(path "/1f58b889-96e6-4877-90a3-5a655db5910b/b9f10619-4e5b-45af-b866-c6815d605ed5/af802241-6422-4666-a084-41c36db8cc4c"
-					(reference "U901")
+					(reference "U1001")
 					(unit 1)
 				)
@@
 		(dnp no)
 		(fields_autoplaced yes)
-		(property "Reference" "C906"
+		(property "Reference" "C1006"
 			(at 182.88 87.6299 0)
 			(effects
@@
 			(project "SMU V1"
 				(path "/1f58b889-96e6-4877-90a3-5a655db5910b/b9f10619-4e5b-45af-b866-c6815d605ed5/af802241-6422-4666-a084-41c36db8cc4c"
-					(reference "C906")
+					(reference "C1006")
 					(unit 1)
 				)
@@
 		(dnp no)
 		(fields_autoplaced yes)
-		(property "Reference" "C901"
+		(property "Reference" "C1001"
 			(at 54.61 87.6299 0)
 			(effects
@@
 			(project "SMU V1"
 				(path "/1f58b889-96e6-4877-90a3-5a655db5910b/b9f10619-4e5b-45af-b866-c6815d605ed5/af802241-6422-4666-a084-41c36db8cc4c"
-					(reference "C901")
+					(reference "C1001")
 					(unit 1)
 				)
@@
 		(dnp no)
 		(fields_autoplaced yes)
-		(property "Reference" "R903"
+		(property "Reference" "R1003"
 			(at 232.41 99.0599 90)
 			(effects
@@
 			(project "SMU V1"
 				(path "/1f58b889-96e6-4877-90a3-5a655db5910b/b9f10619-4e5b-45af-b866-c6815d605ed5/af802241-6422-4666-a084-41c36db8cc4c"
-					(reference "R903")
+					(reference "R1003")
 					(unit 1)
 				)
@@
 		(dnp no)
 		(fields_autoplaced yes)
-		(property "Reference" "C902"
+		(property "Reference" "C1002"
 			(at 67.31 87.6299 0)
 			(effects
@@
 			(project "SMU V1"
 				(path "/1f58b889-96e6-4877-90a3-5a655db5910b/b9f10619-4e5b-45af-b866-c6815d605ed5/af802241-6422-4666-a084-41c36db8cc4c"
-					(reference "C902")
+					(reference "C1002")
 					(unit 1)
 				)
@@
 		(dnp no)
 		(fields_autoplaced yes)
-		(property "Reference" "C907"
+		(property "Reference" "C1007"
 			(at 195.58 87.6299 0)
 			(effects
@@
 			(project "SMU V1"
 				(path "/1f58b889-96e6-4877-90a3-5a655db5910b/b9f10619-4e5b-45af-b866-c6815d605ed5/af802241-6422-4666-a084-41c36db8cc4c"
-					(reference "C907")
+					(reference "C1007")
 					(unit 1)
 				)
@@
 		(dnp no)
 		(fields_autoplaced yes)
-		(property "Reference" "C905"
+		(property "Reference" "C1005"
 			(at 170.18 87.6299 0)
 			(effects
@@
 			(project "SMU V1"
 				(path "/1f58b889-96e6-4877-90a3-5a655db5910b/b9f10619-4e5b-45af-b866-c6815d605ed5/af802241-6422-4666-a084-41c36db8cc4c"
-					(reference "C905")
+					(reference "C1005")
 					(unit 1)
 				)
@@
 		(dnp no)
 		(fields_autoplaced yes)
-		(property "Reference" "#PWR0901"
+		(property "Reference" "#PWR01001"
 			(at 92.71 114.3 0)
 			(effects
@@
 			(project "SMU V1"
 				(path "/1f58b889-96e6-4877-90a3-5a655db5910b/b9f10619-4e5b-45af-b866-c6815d605ed5/af802241-6422-4666-a084-41c36db8cc4c"
-					(reference "#PWR0901")
+					(reference "#PWR01001")
 					(unit 1)
 				)
@@
 		(dnp no)
 		(fields_autoplaced yes)
-		(property "Reference" "R901"
+		(property "Reference" "R1001"
 			(at 107.95 60.96 0)
 			(effects
@@
 			(project ""
 				(path "/1f58b889-96e6-4877-90a3-5a655db5910b/b9f10619-4e5b-45af-b866-c6815d605ed5/af802241-6422-4666-a084-41c36db8cc4c"
-					(reference "R901")
+					(reference "R1001")
 					(unit 1)
 				)
@@
 		(dnp no)
 		(fields_autoplaced yes)
-		(property "Reference" "C908"
+		(property "Reference" "C1008"
 			(at 208.28 87.6299 0)
 			(effects
@@
 			(project "SMU V1"
 				(path "/1f58b889-96e6-4877-90a3-5a655db5910b/b9f10619-4e5b-45af-b866-c6815d605ed5/af802241-6422-4666-a084-41c36db8cc4c"
-					(reference "C908")
+					(reference "C1008")
 					(unit 1)
 				)
