File: SMU V2/Antenna1.kicad_sch (KiCad schematic)
At the start: 9 parts, among them J1101 SMA

Commit message: v2 layout
Changed lines of the file:
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@@
 	)
 	(hierarchical_label "GPS1_ANTENNA_RF"
-		(shape output)
+		(shape bidirectional)
 		(at 110.49 85.09 180)
 		(effects
