File: SMU V2/Microcontroller.kicad_sch (KiCad schematic)
At the start: 9 parts

Commit message: v2
Parts:
- removed MCU201: Krill, bfr_connectors:TE_1-2199119-5, symbol bfr_microcontrollers:Krill
- removed R201, R202: 0, Resistor_SMD:R_0603_1608Metric_Pad0.98x0.95mm_HandSolder, symbol bfr_resistors:RMCF0603ZT0R00
- added MCU201: Krill, bfr_connectors:Krill, symbol bfr_microcontroller_breakouts:Krill
- TP201: renamed from TP205; value CANH -> SMD Test Point
- TP202: renamed from TP206; value CANL -> SMD Test Point
Connections:
- net +5V: now also MCU201.67 (5V), MCU201.69 (5V), MCU201.71 (5V)
- net CAN+: now also MCU201.1 (MCU_CAN+)
- net CAN-: now also MCU201.3 (MCU_CAN-)
- net GND: now also MCU201.10 (GND), MCU201.11 (GND), MCU201.14 (GND), MCU201.15 (GND), MCU201.18 (GND), MCU201.19 (GND), MCU201.2 (GND), MCU201.22 (GND), MCU201.23 (GND), MCU201.26 (GND), MCU201.27 (GND), MCU201.30 (GND), MCU201.31 (GND), MCU201.34 (GND), MCU201.35 (GND), MCU201.38 (GND), MCU201.39 (GND), MCU201.4 (GND), MCU201.42 (GND), MCU201.43 (GND), MCU201.46 (GND), MCU201.47 (GND), MCU201.5 (GND), MCU201.50 (GND), MCU201.51 (GND), MCU201.54 (GND), MCU201.55 (GND), MCU201.57 (GND), MCU201.6 (GND), MCU201.7 (GND), MCU201.73 (GND), MCU201.75 (GND)
- net GPS_UART.RX: now also MCU201.40 (PB10)
- net GPS_UART.TX: now also MCU201.36 (PB11)
- net IMU_SPI.CS: now also MCU201.45 (PA4)
- net IMU_SPI.MISO: now also MCU201.37 (PA6)
- net IMU_SPI.MOSI: now also MCU201.33 (PA7)
- net IMU_SPI.SCK: now also MCU201.41 (PA5)
- new net: MCU201.70 (3V3A), MCU201.72 (3V3A), MCU201.74 (3V3A)
- new net GPS_PGOOD: MCU201.8 (PB5)
- new net IMU_INT1: MCU201.29 (PA8)
- new net IMU_INT2: MCU201.25 (PA9)
- no-connect marks 20 -> 14

Commit message: v2 layout
Parts:
- removed TP201, TP202: SMD Test Point, bfr_utilities:TestPoint_Keystone_5019_Miniature, symbol bfr_utilities:SMD_Test_Point
Connections:
- net GPS1.UART_RX: now reaches MCU201.12 (PB6)
- net GPS1.UART_TX: now reaches MCU201.16 (PB7)
- net DISP_I2C_SDA: now reaches MCU201.24 (PB14)
- net DISP_I2C_SCL: now reaches MCU201.28 (PB13)
- net GPS2.ANT_ON: now reaches MCU201.32 (PB12)
- net GPS1.1PPS: now reaches MCU201.44 (PB2)
- net GPS1.RST: now reaches MCU201.48 (PB1)
- net GPS1.ANT_ON: now reaches MCU201.52 (PB0)
- net GPS2.1PPS: now reaches MCU201.13 (PA12)
- net GPS2.RST: now reaches MCU201.17 (PA11)
- net GPS2.WKUP: now reaches MCU201.9 (PA15)
- net GPS_PGOOD renamed GPS1.WKUP
- net GPS_UART.RX renamed GPS2.UART_RX
- net GPS_UART.TX renamed GPS2.UART_TX
- no-connect marks 14 -> 8
Other:
- moved on the sheet: C201, C202, C203, C204, MCU201A, MCU201B, MCU201C
