File: SMU V2/SMU V2.kicad_pcb (KiCad board)
At the start: 4 copper layers, 75 parts, among them J1001 SMA, J401 Connector, J402 Connector, Q1101 SI2301CDS-T1-GE3, U601 LSM6DSOTR, U701 TPS7A2033PDBVR, U801 TPS7A2033PDBVR, U901 TPS5430DDAR, U902 ETQ-P3M150KVN

Commit message: v2 layout
Parts:
- removed C903: 1.8p, Capacitor_SMD:C_0805_2012Metric_Pad1.18x1.45mm_HandSolder
- removed C904: 10n, Capacitor_SMD:C_0603_1608Metric_Pad1.08x0.95mm_HandSolder
- removed C905, C906, C907, C908, C909: 100u, Capacitor_SMD:C_1206_3216Metric_Pad1.33x1.80mm_HandSolder
- removed D1101: Green, Diode_SMD:D_0805_2012Metric_Pad1.15x1.40mm_HandSolder
- removed F1101: 500mA, Fuse:Fuse_1812_4532Metric
- removed J1001: SMA, bfr_connectors:THT SMA
- removed L1001: 68n, Inductor_SMD:L_0402_1005Metric_Pad0.77x0.64mm_HandSolder
- removed Q1101: SI2301CDS-T1-GE3, Package_TO_SOT_SMD:SOT-23-3
- removed R701, R801: 100k, Resistor_SMD:R_0402_1005Metric_Pad0.72x0.64mm_HandSolder
- removed R901: 180k, Resistor_SMD:R_0805_2012Metric_Pad1.20x1.40mm_HandSolder
- removed R903: 3.3k, Resistor_SMD:R_0402_1005Metric_Pad0.72x0.64mm_HandSolder
- removed TP201, TP202, TP302, TP303, TP304, TP305, TP306, TP307, TP601, TP602, TP603, TP604, TP605, TP606, TP607: SMD Test Point, bfr_utilities:TestPoint_Keystone_5019_Miniature
- removed TVS1101: 16Vrwm, Diode_SMD:D_SMA-SMB_Universal_Handsoldering
- removed U902: ETQ-P3M150KVN, bfr_inductors:BWVS005050404R7M00
- added C1006: 100u, Capacitor_SMD:C_1206_3216Metric_Pad1.33x1.80mm_HandSolder, F.Cu at (161.4, 133.9)
- added C1007: 100u, Capacitor_SMD:C_1206_3216Metric_Pad1.33x1.80mm_HandSolder, F.Cu at (161.4, 131.4)
- added C1008: 100u, Capacitor_SMD:C_1206_3216Metric_Pad1.33x1.80mm_HandSolder, F.Cu at (161.4, 128.9)
- added C1009: 100u, Capacitor_SMD:C_1206_3216Metric_Pad1.33x1.80mm_HandSolder, F.Cu at (161.3, 126.4)
- added C1101: 100n, Capacitor_SMD:C_0402_1005Metric_Pad0.74x0.62mm_HandSolder, F.Cu at (172.9, 76.1)
- added C1102: 100p, Capacitor_SMD:C_0402_1005Metric_Pad0.74x0.62mm_HandSolder, F.Cu at (187.9, 76.6)
- added C1103: 100p, Capacitor_SMD:C_0402_1005Metric_Pad0.74x0.62mm_HandSolder, F.Cu at (174.1, 76.1)
- added C1104: 100p, Capacitor_SMD:C_0402_1005Metric_Pad0.74x0.62mm_HandSolder, F.Cu at (187.9, 75.6)
- added C1105: 100p, Capacitor_SMD:C_0402_1005Metric_Pad0.74x0.62mm_HandSolder, F.Cu at (185.5, 75.5)
- added C1201: 100n, Capacitor_SMD:C_0402_1005Metric_Pad0.74x0.62mm_HandSolder, F.Cu at (134.0, 67.8)
- added C1202: 100p, Capacitor_SMD:C_0402_1005Metric_Pad0.74x0.62mm_HandSolder, F.Cu at (123.3, 68.3)
- added C1203: 100p, Capacitor_SMD:C_0402_1005Metric_Pad0.74x0.62mm_HandSolder, F.Cu at (134.0, 68.9)
- added C1204: 100p, Capacitor_SMD:C_0402_1005Metric_Pad0.74x0.62mm_HandSolder, F.Cu at (122.1, 68.3)
- added C1205: 100p, Capacitor_SMD:C_0402_1005Metric_Pad0.74x0.62mm_HandSolder, F.Cu at (122.6, 66.7)
- added C1401: 10u, Capacitor_SMD:C_0603_1608Metric_Pad1.08x0.95mm_HandSolder, F.Cu at (154.8, 124.1)
- added C1402: 10u, Capacitor_SMD:C_0603_1608Metric_Pad1.08x0.95mm_HandSolder, F.Cu at (154.8, 125.7)
- added C1403: 10u, Capacitor_SMD:C_0603_1608Metric_Pad1.08x0.95mm_HandSolder, F.Cu at (154.8, 127.3)
- added C1404: 10u, Capacitor_SMD:C_0603_1608Metric_Pad1.08x0.95mm_HandSolder, F.Cu at (154.8, 128.9)
- added C504: 100n, Capacitor_SMD:C_0402_1005Metric_Pad0.74x0.62mm_HandSolder, F.Cu at (135.9, 92.8)
- added C505: 4.7u, Capacitor_SMD:C_0603_1608Metric_Pad1.08x0.95mm_HandSolder, F.Cu at (175.2, 97.4)
- added C506: 4.7u, Capacitor_SMD:C_0603_1608Metric_Pad1.08x0.95mm_HandSolder, F.Cu at (137.3, 93.3)
- added D1001: 550m, Diode_SMD:D_SMA_Handsoldering, F.Cu at (175.9, 130.0)
- added D1201: Green, Diode_SMD:D_0805_2012Metric_Pad1.15x1.40mm_HandSolder, F.Cu at (180.7, 133.8)
- added D1401: Green, Diode_SMD:D_0805_2012Metric_Pad1.15x1.40mm_HandSolder, F.Cu at (148.5, 122.1)
- added F1201: 500mA, Fuse:Fuse_1812_4532Metric, F.Cu at (180.3, 128.2)
- added GPS502: LC29HEAMD, bfr_sensors:Quectel LC49, F.Cu at (180.7, 87.8)
- added J1101: SMA, bfr_connectors:THT SMA, F.Cu at (180.2, 73.8)
- added J1201: SMA, bfr_connectors:THT SMA, F.Cu at (128.0, 66.4)
- added L1101: 68n, Inductor_SMD:L_0402_1005Metric_Pad0.77x0.64mm_HandSolder, F.Cu at (173.4, 74.3)
- added L1201: 68n, Inductor_SMD:L_0402_1005Metric_Pad0.77x0.64mm_HandSolder, F.Cu at (134.1, 66.8)
- added Q1201: SI2301CDS-T1-GE3, Package_TO_SOT_SMD:SOT-23-3, F.Cu at (186.1, 130.6)
- added R1003: 3.3k, Resistor_SMD:R_0402_1005Metric_Pad0.72x0.64mm_HandSolder, F.Cu at (165.1, 131.2)
- added R1102: 0, Resistor_SMD:R_0402_1005Metric_Pad0.72x0.64mm_HandSolder, F.Cu at (185.5, 76.6)
- added R1201: 1.8k, Resistor_SMD:R_0603_1608Metric_Pad0.98x0.95mm_HandSolder, F.Cu at (180.6, 132.0)
- added R1202: 10, Resistor_SMD:R_0402_1005Metric_Pad0.72x0.64mm_HandSolder, F.Cu at (134.0, 70.0)
- added R1203: 0, Resistor_SMD:R_0402_1005Metric_Pad0.72x0.64mm_HandSolder, F.Cu at (122.7, 70.0)
- added R1301: 4.7k, Resistor_SMD:R_0402_1005Metric_Pad0.72x0.64mm_HandSolder, F.Cu at (135.6, 117.3)
- added R1302: 4.7k, Resistor_SMD:R_0402_1005Metric_Pad0.72x0.64mm_HandSolder, F.Cu at (135.6, 114.7)
- added R1401: 220, Resistor_SMD:R_0402_1005Metric_Pad0.72x0.64mm_HandSolder, F.Cu at (145.4, 122.5)
- added TVS1201: 16Vrwm, Diode_SMD:D_SMA-SMB_Universal_Handsoldering, F.Cu at (188.4, 126.5)
- added U1001: TPS5430DDAR, Package_SO:TI_SO-PowerPAD-8, F.Cu at (169.8, 132.2)
- added U1002: ETQ-P3M150KVN, bfr_inductors:BWVS005050404R7M00, F.Cu at (169.8, 126.4)
- added U1301: Display, bfr_utilities:1.3 OLED Display, F.Cu at (120.0, 114.6)
- added U1401: AMS1117-3.3, Package_TO_SOT_SMD:SOT-223-3_TabPin2, F.Cu at (148.6, 126.7)
- C1001: value 100n -> 22u; footprint Capacitor_SMD:C_0402_1005Metric_Pad0.74x0.62mm_HandSolder -> Capacitor_SMD:C_0603_1608Metric_Pad1.08x0.95mm_HandSolder
- C1002: value 100p -> 22u; footprint Capacitor_SMD:C_0402_1005Metric_Pad0.74x0.62mm_HandSolder -> Capacitor_SMD:C_0603_1608Metric_Pad1.08x0.95mm_HandSolder
- C1003: value 100p -> 1.8p; footprint Capacitor_SMD:C_0402_1005Metric_Pad0.74x0.62mm_HandSolder -> Capacitor_SMD:C_0805_2012Metric_Pad1.18x1.45mm_HandSolder
- C1004: value 100p -> 10n; footprint Capacitor_SMD:C_0402_1005Metric_Pad0.74x0.62mm_HandSolder -> Capacitor_SMD:C_0603_1608Metric_Pad1.08x0.95mm_HandSolder
- C1005: value 100p -> 100u; footprint Capacitor_SMD:C_0402_1005Metric_Pad0.74x0.62mm_HandSolder -> Capacitor_SMD:C_1206_3216Metric_Pad1.33x1.80mm_HandSolder
- C502: value 100n -> 33p
- C503: value 4.7u -> 100n; footprint Capacitor_SMD:C_0603_1608Metric_Pad1.08x0.95mm_HandSolder -> Capacitor_SMD:C_0402_1005Metric_Pad0.74x0.62mm_HandSolder
- C901, C902: value 22u -> 2.2u; footprint Capacitor_SMD:C_0603_1608Metric_Pad1.08x0.95mm_HandSolder -> Capacitor_SMD:C_0402_1005Metric_Pad0.74x0.62mm_HandSolder
- D901: value 550m -> Green; footprint Diode_SMD:D_SMA_Handsoldering -> Diode_SMD:D_0805_2012Metric_Pad1.15x1.40mm_HandSolder
- R1001: value 10 -> 180k; footprint Resistor_SMD:R_0402_1005Metric_Pad0.72x0.64mm_HandSolder -> Resistor_SMD:R_0805_2012Metric_Pad1.20x1.40mm_HandSolder
- R1002: value 0 -> 10k
- R1101: value 1.8k -> 10; footprint Resistor_SMD:R_0603_1608Metric_Pad0.98x0.95mm_HandSolder -> Resistor_SMD:R_0402_1005Metric_Pad0.72x0.64mm_HandSolder
- R902: value 10k -> 120; footprint Resistor_SMD:R_0402_1005Metric_Pad0.72x0.64mm_HandSolder -> Resistor_SMD:R_0603_1608Metric_Pad0.98x0.95mm_HandSolder
- TP301: moved to B.Cu
- U901: value TPS5430DDAR -> TPS7A2033PDBVR; footprint Package_SO:TI_SO-PowerPAD-8 -> Package_TO_SOT_SMD:SOT-23-5_HandSoldering
- moved C1001 80.4 mm to (171.3, 138.5), turned to 180 degrees
- moved C1002 76.9 mm to (171.3, 136.9), turned to 180 degrees
- moved C1003 75.4 mm to (174.2, 137.9), turned to -90 degrees
- moved C802 74.1 mm to (129.7, 92.0), turned to -90 degrees
- moved C1004 73.8 mm to (167.7, 136.9)
- moved C1005 73.4 mm to (161.4, 136.4), turned to 180 degrees
- moved C401 72.5 mm to (188.4, 118.6)
- moved J401 72.2 mm to (185.8, 119.7)
- moved C402 72.0 mm to (190.6, 118.6)
- moved R1001 71.4 mm to (167.7, 138.6)
- moved R802 71.2 mm to (132.5, 89.3)
- moved C801 68.4 mm to (135.4, 94.5)
- moved U801 66.9 mm to (132.3, 92.7), turned to 90 degrees
- moved R1002 65.7 mm to (165.1, 133.6), turned to -90 degrees
- moved D801 62.9 mm to (136.2, 90.6), turned to 180 degrees
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Connections:
- net /GPS_UART.TX renamed /GPS2.UART_TX
- C1001 pad 1: /Antenna/GPS_RF_VDD_R -> /Power/5V Buck/PPVAR_VBATT_PROT
- C1002 pad 1: /Antenna/GPS_ANT_RF -> /Power/5V Buck/PPVAR_VBATT_PROT
- C1003 pad 1: /Antenna/GPS_RF_VDD_R -> /Power/5V Buck/PPVAR_VBATT_PROT
- C1003 pad 2: GND -> /Power/5V Buck/Rsnub
- C1004 pad 1: /Antenna/GPS_ANT_RF_R -> Net-(U1001-BOOT)
- C1004 pad 2: GND -> /Power/5V Buck/SWITCH_NODE
- C1005 pad 1: /Antenna/GPS_ANT_RF_R -> +5V
- C1005 pad 2: /Antenna/ANT_OUT_RF -> GND
- C501 pad 1: /GPS/PP3300_GPS_VCC -> /GPS/PP3300_GPS1_VCC
- C502 pad 1: /GPS/PP3300_GPS_VCC -> /GPS/PP3300_GPS2_VCC
- C503 pad 1: /GPS/PP3300_GPS_VCC -> /GPS/PP3300_GPS1_VCC
- C702 pad 1: /GPS/PP3300_GPS_VCC -> /GPS/PP3300_GPS1_VCC
- C802 pad 1: /IMU/PP3300_IMU_VDD -> /GPS/PP3300_GPS2_VCC
- C901 pad 1: /Power/5V Buck/PPVAR_VBATT_PROT -> +5V
- C902 pad 1: /Power/5V Buck/PPVAR_VBATT_PROT -> /IMU/PP3300_IMU_VDD
- D901 pad 1: /Power/5V Buck/SWITCH_NODE -> GND
- D901 pad 2: GND -> Net-(D901-A)
- GPS501 pad 1: /GPS_WKUP -> /GPS2.WKUP
- GPS501 pad 11: /Antenna/GPS_ANT_RF -> /GPS2_ANTENNA_RF
- GPS501 pad 14: /GPS_ANT_ON -> /GPS2.ANT_ON
- GPS501 pad 21: /GPS_UART.RX -> /GPS1.UART_TX
- GPS501 pad 22: /GPS/PP3300_GPS_VCC -> /GPS/PP3300_GPS2_VCC
- GPS501 pad 23: /GPS/PP3300_GPS_VCC -> /GPS/PP3300_GPS2_VCC
- GPS501 pad 3: /GPS_1PPS -> /GPS2.1PPS
- GPS501 pad 8: /GPS_~{RST} -> /GPS2.RST
- GPS501 pad 9: /Antenna/GPS_RF_VDD -> /Antenna2/GPS2_RF_VDD
- MCU201 pad 12: /GPS_1PPS -> /GPS1.UART_RX
- MCU201 pad 13: unconnected-(MCU201A-PA12-Pad13) -> /GPS2.1PPS
- MCU201 pad 16: /GPS_WKUP -> /GPS1.UART_TX
- MCU201 pad 17: unconnected-(MCU201A-PA11-Pad17) -> /GPS2.RST
- MCU201 pad 24: unconnected-(MCU201B-PB14-Pad24) -> /DISP_I2C_SDA
- MCU201 pad 28: unconnected-(MCU201B-PB13-Pad28) -> /DISP_I2C_SCL
- MCU201 pad 32: unconnected-(MCU201B-PB12-Pad32) -> /GPS2.ANT_ON
- MCU201 pad 40: /GPS_UART.RX -> /GPS1.UART_TX
- MCU201 pad 44: /GPS_ANT_ON -> /GPS1.1PPS
- MCU201 pad 48: /GPS_LDO_EN -> /GPS1.RST
- MCU201 pad 52: /GPS_~{RST} -> /GPS1.ANT_ON
- MCU201 pad 8: /GPS_PGOOD -> /GPS1.WKUP
- MCU201 pad 9: unconnected-(MCU201A-PA15-Pad9) -> /GPS2.WKUP
- R1001 pad 1: /Antenna/GPS_RF_VDD -> /Power/5V Buck/Rsnub
- R1001 pad 2: /Antenna/GPS_RF_VDD_R -> /Power/5V Buck/SWITCH_NODE
- R1002 pad 1: /Antenna/GPS_ANT_RF -> /Power/5V Buck/BUCK_VSENSE
- R1002 pad 2: /Antenna/GPS_ANT_RF_R -> +5V
- R1101 pad 1: /Power/5V Buck/PPVAR_VBATT_PROT -> /Antenna1/GPS1_RF_VDD
- R1101 pad 2: Net-(D1101-A) -> /Antenna1/GPS1_RF_VDD_R
- R702 pad 1: /GPS/PP3300_GPS_VCC -> /GPS/PP3300_GPS1_VCC
- R802 pad 1: /IMU/PP3300_IMU_VDD -> /GPS/PP3300_GPS2_VCC
- R902 pad 1: /Power/5V Buck/BUCK_VSENSE -> /IMU/PP3300_IMU_VDD
- R902 pad 2: +5V -> Net-(D901-A)
- TP301 pad 1: /Main IO/VBATT+ -> GND
- U701 pad 3: /GPS_LDO_EN -> +5V
- U701 pad 5: /GPS/PP3300_GPS_VCC -> /GPS/PP3300_GPS1_VCC
- U801 pad 3: /IMU/GPS Power/LDO_EN -> +5V
- U801 pad 5: /IMU/PP3300_IMU_VDD -> /GPS/PP3300_GPS2_VCC
- U901 pad 1: Net-(U901-BOOT) -> +5V
- U901 pad 2: unconnected-(U901-NC-Pad2) -> GND
- U901 pad 3: unconnected-(U901-NC-Pad3) -> +5V
- U901 pad 4: /Power/5V Buck/BUCK_VSENSE -> unconnected-(U901-NC-Pad4)
- U901 pad 5: unconnected-(U901-EN-Pad5) -> /IMU/PP3300_IMU_VDD
Routing:
- net /CAN+: track 0.00 -> 111.9 mm
- net /CAN-: track 0.00 -> 107.3 mm
- net /DISP_I2C_SCL: track 0.00 -> 84.0 mm, vias 0 -> 2
- net /Main IO/VBATT+: track 0.00 -> 81.7 mm
- net GND: track 0.00 -> 78.5 mm, vias 0 -> 29
- net /DISP_I2C_SDA: track 0.00 -> 77.0 mm, vias 0 -> 2
- net +5V: track 0.00 -> 70.2 mm, vias 0 -> 11
- net /GPS1.UART_TX: track 0.00 -> 65.0 mm
- net /GPS1.WKUP: track 0.00 -> 53.8 mm, vias 0 -> 2
- net +3V3: track 0.00 -> 46.6 mm
- net /GPS2.UART_TX: track 0.00 -> 41.4 mm
- net /GPS2.ANT_ON: track 0.00 -> 41.4 mm, vias 0 -> 2
- net /GPS1.1PPS: track 0.00 -> 40.3 mm
- net /GPS1.RST: track 0.00 -> 37.2 mm
- net /GPS1.UART_RX: track 0.00 -> 35.6 mm, vias 0 -> 2
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- added copper zone on In2.Cu, net +5V
- added copper zone on B.Cu, net GND
- added copper zone on F.Cu, net GND
- added copper zone on In1.Cu, net GND
Other:
- board outline added: 94.8 x 90.7 mm

Commit message: test
Parts:
- removed R1301, R1302: 4.7k, Resistor_SMD:R_0402_1005Metric_Pad0.72x0.64mm_HandSolder
- removed U1301: Display, bfr_utilities:1.3 OLED Display
- moved TVS1201 58.6 mm to (130.8, 115.6), turned to 180 degrees
- moved C1104 56.8 mm to (132.3, 87.0), turned to 90 degrees
- moved Q1201 56.3 mm to (133.1, 111.4), turned to 180 degrees
- moved C1102 55.6 mm to (133.3, 87.0), turned to 90 degrees
- moved C1105 55.0 mm to (132.2, 89.4), turned to -90 degrees
- moved J1101 53.9 mm to (130.5, 94.7), turned to 0 degrees
- moved R1102 53.7 mm to (133.3, 89.4), turned to 90 degrees
- moved L1101 50.3 mm to (131.0, 101.5), turned to 90 degrees
- moved R1101 50.0 mm to (131.7, 99.7), turned to 180 degrees
- moved D1201 49.4 mm to (138.5, 108.2), turned to 180 degrees
- moved C1103 48.1 mm to (132.8, 100.8), turned to 0 degrees
- moved J401 47.8 mm to (168.9, 75.0), turned to -90 degrees
- moved C1101 47.8 mm to (132.8, 102.0), turned to 0 degrees
- moved R1201 47.4 mm to (138.6, 110.0), turned to 180 degrees
- moved C401 46.9 mm to (165.2, 77.8), turned to 0 degrees
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Connections:
- net /GPS1.UART_TX renamed /GPS2.UART_RX
- MCU201 pad 24: /DISP_I2C_SDA -> /Microcontroller/DISP_I2C_SDA
- MCU201 pad 28: /DISP_I2C_SCL -> /Microcontroller/DISP_I2C_SCL
Routing:
- net /DISP_I2C_SCL: track 84.0 -> 0.00 mm, vias 2 -> 0
- net /DISP_I2C_SDA: track 77.0 -> 0.00 mm, vias 2 -> 0
- net /CAN+: track 111.9 -> 66.0 mm, vias 0 -> 1
- net /CAN-: track 107.3 -> 64.4 mm, vias 0 -> 1
- net /Main IO/VBATT+: track 81.7 -> 120.8 mm, vias 0 -> 10
- net /GPS1.ANT_ON: track 21.4 -> 56.6 mm, vias 0 -> 2
- net +3V3: track 46.6 -> 14.8 mm
- net /GPS1.WKUP: track 53.8 -> 35.2 mm
- net /GPS2.RST: track 34.8 -> 17.9 mm
- net /GPS1.1PPS: track 40.3 -> 23.6 mm, vias 0 -> 2
- net /GPS2.UART_TX: track 41.4 -> 25.0 mm, vias 0 -> 4
- net /GPS2.ANT_ON: track 41.4 -> 26.7 mm, vias 2 -> 0
- net GND: track 78.5 -> 70.9 mm, vias 29 -> 116
- net /GPS1.RST: track 37.2 -> 31.3 mm, vias 0 -> 2
- net /GPS2.UART_RX: track 65.0 -> 59.1 mm, vias 0 -> 2
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- added copper zone on B.Cu, net /Main IO/VBATT+
- added copper zone on F.Cu, net /Main IO/VBATT+
Other:
- board size 94.8 x 90.7 mm -> 53.4 x 72.2 mm
