File: SMU V2/SMU V2.kicad_sch (KiCad schematic)
At the start: 0 parts

Commit message: v2 layout
Other:
- sheet Antenna renamed Antenna1
- added sheet Antenna2 (Antenna2.kicad_sch)
- added sheet Display (Display.kicad_sch)
- sheet Antenna1: file antenna.kicad_sch -> Antenna1.kicad_sch
- sheet Antenna1 ports: added GPS1_ANTENNA_RF, GPS1_RF_VDD; removed GPS_ANTENNA_RF, GPS_RF_VDD
- sheet GPS ports: added GPS1_ANTENNA_RF, GPS1_RF_VDD, GPS2, GPS2_ANTENNA_RF, GPS2_RF_VDD; removed GPS_ANTENNA_RF, GPS_PGOOD, GPS_RF_VDD
- sheet Microcontroller ports: added DISP_I2C, GPS2; removed GPS_PGOOD
- sheet Power ports: added 3V3; removed none

Commit message: test
Connections:
- no-connect marks 0 -> 1
Other:
- removed sheet Display
