File: SMU V2/gps.kicad_sch (KiCad schematic)
At the start: 10 parts

Commit message: v2
Parts:
- removed GPS501: LC29HEAMD, bfr_sensors:Quectel LC49, symbol bfr_utilities:LC29HEAMD
- removed TP501: GPS_UART_RX, bfr_utilities:TestPoint_Keystone_5019_Miniature, symbol bfr_utilities:SMD_Test_Point
- removed TP502: GPS_UART_TX, bfr_utilities:TestPoint_Keystone_5019_Miniature, symbol bfr_utilities:SMD_Test_Point
- removed TP503: GPS_WKUP, bfr_utilities:TestPoint_Keystone_5019_Miniature, symbol bfr_utilities:SMD_Test_Point
- removed TP504: GPS_1PPS, bfr_utilities:TestPoint_Keystone_5019_Miniature, symbol bfr_utilities:SMD_Test_Point
- removed TP505: GPS_nRST, bfr_utilities:TestPoint_Keystone_5019_Miniature, symbol bfr_utilities:SMD_Test_Point
- removed TP506: GPS_+3V3, bfr_utilities:TestPoint_Keystone_5019_Miniature, symbol bfr_utilities:SMD_Test_Point
- added C?: 4.7u, Capacitor_SMD:C_0603_1608Metric_Pad1.08x0.95mm_HandSolder, symbol bfr_capacitors:CL10A475KO8NNNC
- added C?: 33p, Capacitor_SMD:C_0402_1005Metric_Pad0.74x0.62mm_HandSolder, symbol bfr_capacitors:0402CG330J500NT
- added C?: 100n, Capacitor_SMD:C_0402_1005Metric_Pad0.74x0.62mm_HandSolder, symbol bfr_capacitors:CL05B104KO5NNNC
- added GPS? (x4): LC29HEAMD, bfr_sensors:Quectel LC49, symbol bfr_sensors:LC29HEAMD
- renumbered C501 to C?, C503 to C?, C502 to C?
Connections:
- net GND: now also C?.2, C?.2, C?.2, GPS?.10 (GND), GPS?.12 (GND), GPS?.13 (GND), GPS?.15 (RESERVED), GPS?.16 (RESERVED), GPS?.17 (RESERVED), GPS?.18 (RESERVED), GPS?.19 (RESERVED), GPS?.2 (RESERVED), GPS?.24 (GND), GPS?.24 (GND), GPS?.4 (RESERVED), GPS?.5 (RESERVED), GPS?.6 (RESERVED)
- net GPS_ANTENNA_RF: now also GPS?.11 (RF_IN)
- net GPS_RF_VDD: now also GPS?.9 (VDD_RF)
- net PP3300_GPS_VCC renamed PP3300_GPS1_VCC
- net PP3300_GPS1_VCC: now also GPS?.22 (V_BCKUP), GPS?.23 (VCC)
- new net: GPS?.15 (RESERVED), GPS?.16 (RESERVED), GPS?.17 (RESERVED), GPS?.18 (RESERVED), GPS?.19 (RESERVED), GPS?.2 (RESERVED), GPS?.4 (RESERVED), GPS?.5 (RESERVED), GPS?.6 (RESERVED) (x2)
- new net GPS1.1PPS: GPS?.3 (1PPS)
- new net GPS1.RST: GPS?.8 (RESET_N)
- new net GPS1.UART_RX: GPS?.21 (UART_RXD)
- new net GPS1.UART_TX: GPS?.20 (UART_TXD), GPS?.21 (UART_RXD)
- new net GPS1.WKUP: GPS?.1 (WAKEUP)
- new net GPS2.1PPS: GPS?.3 (1PPS)
- new net GPS2.ANT_ON: GPS?.14 (ANT_ON)
- new net GPS2.RST: GPS?.8 (RESET_N)
- new net GPS2.UART_TX: GPS?.20 (UART_TXD)
- new net GPS2.WKUP: GPS?.1 (WAKEUP)
- new net PP3300_GPS2_VCC: C?.1, C?.1, C?.1, GPS?.22 (V_BCKUP), GPS?.23 (VCC)
- no-connect marks 2 -> 4
Other:
- added sheet GPS LDO1 (low_noise_ldo.kicad_sch)
- sheet GPS LDO ports: added GPS_PGOOD; removed LDO_EN
- moved on the sheet: C?

Commit message: v2 layout
Parts:
- removed GPS? (x3): LC29HEAMD, bfr_sensors:Quectel LC49, symbol bfr_sensors:LC29HEAMD
- added GPS501: LC29HEAMD, bfr_sensors:Quectel LC49, symbol bfr_sensors:LC29HEAMD
- added unit 2 of GPS502
- gave numbers to parts that had none: 7
Connections:
- net GND: now also GPS501.10 (GND), GPS501.12 (GND), GPS501.13 (GND), GPS501.24 (GND), GPS502.10 (GND), GPS502.12 (GND), GPS502.13 (GND)
- net GPS1.1PPS: now also GPS502.3 (1PPS)
- net GPS1.ANT_ON: now also GPS502.14 (ANT_ON)
- net GPS1.RST: now also GPS502.8 (RESET_N)
- net GPS1.UART_RX: now also GPS502.21 (UART_RXD)
- net GPS1.UART_TX: now also GPS502.20 (UART_TXD), GPS501.21 (UART_RXD); no longer GPS502.21 (UART_RXD)
- net GPS1.WKUP: now also GPS502.1 (WAKEUP)
- net GPS2.1PPS: now also GPS501.3 (1PPS); no longer GPS502.3 (1PPS)
- net GPS2.ANT_ON: now also GPS501.14 (ANT_ON)
- net GPS2.RST: now also GPS501.8 (RESET_N); no longer GPS502.8 (RESET_N)
- net GPS2.UART_TX: now also GPS501.20 (UART_TXD); no longer GPS502.20 (UART_TXD)
- net GPS2.WKUP: now also GPS501.1 (WAKEUP); no longer GPS502.1 (WAKEUP)
- net PP3300_GPS1_VCC: now also GPS502.22 (V_BCKUP), GPS502.23 (VCC)
- net PP3300_GPS2_VCC: now also GPS501.22 (V_BCKUP), GPS501.23 (VCC); no longer GPS502.22 (V_BCKUP), GPS502.23 (VCC)
- new net: GPS501.15 (RESERVED), GPS501.16 (RESERVED), GPS501.17 (RESERVED), GPS501.18 (RESERVED), GPS501.19 (RESERVED), GPS501.2 (RESERVED), GPS501.4 (RESERVED), GPS501.5 (RESERVED), GPS501.6 (RESERVED)
- new net GPS1_ANTENNA_RF: GPS502.11 (RF_IN)
- new net GPS1_RF_VDD: GPS502.9 (VDD_RF)
- new net GPS2_ANTENNA_RF: GPS501.11 (RF_IN)
- new net GPS2_RF_VDD: GPS501.9 (VDD_RF)
- no-connect marks 4 -> 6
Other:
- moved on the sheet: C501, C502, C503, C504, C505, C506, GPS502A
