File: SMU V2/imu.kicad_sch (KiCad schematic)
At the start: 10 parts, among them U601 LSM6DSOTR

Commit message: v2
Parts:
- removed U601: LSM6DSOTR, Package_LGA:LGA-14_3x2.5mm_P0.5mm_LayoutBorder3x4y, symbol bfr_utilities:LSM6DSO
- added U601: LSM6DSOTR, Package_LGA:LGA-14_3x2.5mm_P0.5mm_LayoutBorder3x4y, symbol bfr_sensors:LSM6DSO
- TP601: value IMU_+3V3 -> SMD Test Point
- TP602: value IMU_INT2 -> SMD Test Point
- TP603: value IMU_INT1 -> SMD Test Point
- TP604: value IMU_SPI_CS -> SMD Test Point
- TP605: value IMU_SPI_MISO -> SMD Test Point
- TP606: value IMU_SPI_MOSI -> SMD Test Point
- TP607: value IMU_SPI_SCK -> SMD Test Point
Connections:
- net GND: now also U601.2 (SDx), U601.3 (SCx), U601.6 (GND), U601.7 (GND )
- net IMU_INT1: now also U601.4 (INT1)
- net IMU_INT2: now also U601.9 (INT2)
- net IMU_SPI.CS: now also U601.12 (CS)
- net IMU_SPI.MISO: now also U601.1 (I2C_SA0)
- net IMU_SPI.MOSI: now also U601.14 (I2C_SDA)
- net IMU_SPI.SCK: now also U601.13 (I2C_SCL)
- net PP3300_IMU_VDD: now also U601.5 (VDDIO), U601.8 (VDD)
Changed lines of the file:
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@@
+	)
+	(junction
+		(at 123.19 87.63)
+		(diameter 0)
+		(color 0 0 0 0)
 	)
 	(junction
@@
 	(junction
 		(at 92.71 73.66)
-		(diameter 0)
-		(color 0 0 0 0)
-	)
-	(junction
-		(at 123.19 87.63)
 		(diameter 0)
 		(color 0 0 0 0)
@@
 			)
 		)
-		(property "Value" "IMU_SPI_CS"
+		(property "Value" "SMD Test Point"
 			(at 170.18 71.6497 0)
 			(effects
@@
 			)
 		)
-		(property "Value" "IMU_SPI_SCK"
+		(property "Value" "SMD Test Point"
 			(at 207.01 86.8897 0)
 			(effects
@@
 			)
 		)
-		(property "Value" "IMU_INT1"
+		(property "Value" "SMD Test Point"
 			(at 111.76 105.9397 0)
 			(effects
@@
 			)
 		)
-		(property "Value" "IMU_SPI_MOSI"
+		(property "Value" "SMD Test Point"
 			(at 195.58 81.8097 0)
 			(effects
@@
 	)
 	(symbol
+		(lib_id "bfr_sensors:LSM6DSO")
+		(at 137.16 93.98 0)
+		(unit 1)
+		(exclude_from_sim no)
+		(in_bom yes)
+		(on_board yes)
+		(dnp no)
+		(fields_autoplaced yes)
+		(property "Reference" "U601"
+			(at 137.16 64.77 0)
+			(effects
+				(font
+					(size 1.27 1.27)
+				)
+			)
+		)
+		(property "Value" "LSM6DSOTR"
+			(at 137.16 67.31 0)
+			(effects
+				(font
+					(size 1.27 1.27)
+				)
+			)
+		)
+		(property "Footprint" "Package_LGA:LGA-14_3x2.5mm_P0.5mm_LayoutBorder3x4y"
+			(at 137.16 68.58 0)
+			(effects
+				(font
+					(size 1.27 1.27)
+				)
+				(hide yes)
+			)
+		)
+		(property "Datasheet" "https://www.st.com/resource/en/datasheet/lsm6dso.pdf"
+			(at 137.16 68.58 0)
+			(effects
+				(font
+					(size 1.27 1.27)
+				)
+				(hide yes)
+			)
+		)
+		(property "Description" "6DOF IMU, +-2/4/6/8/16G FSR, 1.71-3.6Vcc, SPI/I2C"
+			(at 137.16 68.58 0)
+			(effects
+				(font
+					(size 1.27 1.27)
+				)
+				(hide yes)
+			)
+		)
+		(property "Manufacturer P/N" "LSM6DSOTR"
+			(at 137.16 68.58 0)
+			(effects
+				(font
+					(size 1.27 1.27)
+				)
+				(hide yes)
+			)
+		)
+		(property "Manufacturer" "STMicroelectronics"
+			(at 137.16 68.58 0)
+			(effects
+				(font
+					(size 1.27 1.27)
+				)
+				(hide yes)
+			)
+		)
+		(property "Digikey P/N" "497-18181-2-ND"
+			(at 137.16 68.58 0)
+			(effects
+				(font
+					(size 1.27 1.27)
+				)
+				(hide yes)
+			)
+		)
+		(property "Mouser P/N" "511-LSM6DSOTR"
+			(at 137.16 68.58 0)
+			(effects
+				(font
+					(size 1.27 1.27)
+				)
+				(hide yes)
+			)
+		)
+		(property "LCSC P/N" "C481766"
+			(at 137.16 68.58 0)
+			(effects
+				(font
+					(size 1.27 1.27)
+				)
+				(hide yes)
+			)
+		)
+		(property "JLC Basic Part" "No"
+			(at 137.16 68.58 0)
+			(effects
+				(font
+					(size 1.27 1.27)
+				)
+				(hide yes)
+			)
+		)
+		(property "Order From" "JLC"
+			(at 137.16 68.58 0)
+			(effects
+				(font
+					(size 1.27 1.27)
+				)
+				(hide yes)
+			)
+		)
+		(property "Created By" "Manual Entry"
+			(at 137.16 68.58 0)
+			(effects
+				(font
+					(size 1.27 1.27)
+				)
+				(hide yes)
+			)
+		)
+		(pin "14"
+		)
+		(pin "12"
+		)
+		(pin "8"
+		)
+		(pin "10"
+		)
+		(pin "1"
+		)
+		(pin "7"
+		)
+		(pin "6"
+		)
+		(pin "9"
+		)
+		(pin "4"
+		)
+		(pin "3"
+		)
+		(pin "11"
+		)
+		(pin "2"
+		)
+		(pin "5"
+		)
+		(pin "13"
+		)
+		(instances
+			(project ""
+				(path "/1f58b889-96e6-4877-90a3-5a655db5910b/4cd2b3ee-b9d4-4006-b5a4-98c8a3d3240f"
+					(reference "U601")
+					(unit 1)
+				)
+			)
+		)
+	)
+	(symbol
 		(lib_id "bfr_utilities:SMD_Test_Point")
 		(at 92.71 71.12 0)
@@
 			)
 		)
-		(property "Value" "IMU_+3V3"
+		(property "Value" "SMD Test Point"
 			(at 95.25 71.6497 0)
 			(effects
@@
 			)
 		)
-		(property "Value" "IMU_SPI_MISO"
+		(property "Value" "SMD Test Point"
 			(at 182.88 76.7297 0)
 			(effects
@@
 			)
 		)
-		(property "Value" "IMU_INT2"
+		(property "Value" "SMD Test Point"
 			(at 111.76 97.0497 0)
 			(effects
@@
 				(path "/1f58b889-96e6-4877-90a3-5a655db5910b/4cd2b3ee-b9d4-4006-b5a4-98c8a3d3240f"
 					(reference "TP602")
-					(unit 1)
-				)
-			)
-		)
-	)
-	(symbol
-		(lib_id "bfr_utilities:LSM6DSO")
-		(at 137.16 93.98 0)
-		(unit 1)
-		(exclude_from_sim no)
-		(in_bom yes)
-		(on_board yes)
-		(dnp no)
-		(fields_autoplaced yes)
-		(property "Reference" "U601"
-			(at 137.16 64.77 0)
-			(effects
-				(font
-					(size 1.27 1.27)
-				)
-			)
-		)
-		(property "Value" "LSM6DSOTR"
-			(at 137.16 67.31 0)
-			(effects
-				(font
-					(size 1.27 1.27)
-				)
-			)
-		)
-		(property "Footprint" "Package_LGA:LGA-14_3x2.5mm_P0.5mm_LayoutBorder3x4y"
-			(at 137.16 68.58 0)
-			(effects
-				(font
-					(size 1.27 1.27)
-				)
-				(hide yes)
-			)
-		)
-		(property "Datasheet" "https://www.st.com/resource/en/datasheet/lsm6dso.pdf"
-			(at 137.16 68.58 0)
-			(effects
-				(font
-					(size 1.27 1.27)
-				)
-				(hide yes)
-			)
-		)
-		(property "Description" "6DOF IMU, +-2/4/6/8/16G FSR, 1.71-3.6Vcc, SPI/I2C"
-			(at 137.16 68.58 0)
-			(effects
-				(font
-					(size 1.27 1.27)
-				)
-				(hide yes)
-			)
-		)
-		(property "Manufacturer P/N" "LSM6DSOTR"
-			(at 137.16 68.58 0)
-			(effects
-				(font
-					(size 1.27 1.27)
-				)
-				(hide yes)
-			)
-		)
-		(property "Manufacturer" "STMicroelectronics"
-			(at 137.16 68.58 0)
-			(effects
-				(font
-					(size 1.27 1.27)
-				)
-				(hide yes)
-			)
-		)
-		(property "Digikey P/N" "497-18181-2-ND"
-			(at 137.16 68.58 0)
-			(effects
-				(font
-					(size 1.27 1.27)
-				)
-				(hide yes)
-			)
-		)
-		(property "Mouser P/N" "511-LSM6DSOTR"
-			(at 137.16 68.58 0)
-			(effects
-				(font
-					(size 1.27 1.27)
-				)
-				(hide yes)
-			)
-		)
-		(property "LCSC P/N" "C481766"
-			(at 137.16 68.58 0)
-			(effects
-				(font
-					(size 1.27 1.27)
-				)
-				(hide yes)
-			)
-		)
-		(property "JLC Basic Part" "No"
-			(at 137.16 68.58 0)
-			(effects
-				(font
-					(size 1.27 1.27)
-				)
-				(hide yes)
-			)
-		)
-		(property "Order From" "LCSC"
-			(at 137.16 68.58 0)
-			(effects
-				(font
-					(size 1.27 1.27)
-				)
-				(hide yes)
-			)
-		)
-		(property "Created By" "Manual Entry"
-			(at 137.16 68.58 0)
-			(effects
-				(font
-					(size 1.27 1.27)
-				)
-				(hide yes)
-			)
-		)
-		(property "Pretty Name" ""
-			(at 137.16 93.98 0)
-			(effects
-				(font
-					(size 1.27 1.27)
-				)
-				(hide yes)
-			)
-		)
-		(pin "6"
-		)
-		(pin "1"
-			(alternate "SPI_MISO")
-		)
-		(pin "8"
-		)
-		(pin "7"
-		)
-		(pin "4"
-		)
-		(pin "5"
-		)
-		(pin "9"
-		)
-		(pin "12"
-		)
-		(pin "11"
-		)
-		(pin "10"
-		)
-		(pin "13"
-			(alternate "SPI_SCK")
-		)
-		(pin "3"
-		)
-		(pin "14"
-			(alternate "4W_SPI_MOSI")
-		)
-		(pin "2"
-		)
-		(instances
-			(project ""
-				(path "/1f58b889-96e6-4877-90a3-5a655db5910b/4cd2b3ee-b9d4-4006-b5a4-98c8a3d3240f"
-					(reference "U601")
 					(unit 1)
 				)
@@
 		)
 		(instances
-			(project "SMU V1"
+			(project "SMU V2"
 				(path "/1f58b889-96e6-4877-90a3-5a655db5910b/4cd2b3ee-b9d4-4006-b5a4-98c8a3d3240f"
 					(page "9")

Commit message: v2 layout
Parts:
- removed TP601, TP602, TP603, TP604, TP605, TP606, TP607: SMD Test Point, bfr_utilities:TestPoint_Keystone_5019_Miniature, symbol bfr_utilities:SMD_Test_Point
