File: SMU V2/low_noise_ldo.kicad_sch (KiCad schematic)
At the start: 6 parts

Commit message: v2 layout
Parts:
- removed R?: 100k, Resistor_SMD:R_0402_1005Metric_Pad0.72x0.64mm_HandSolder, symbol bfr_resistors:RMCF0402FT100K
- gave numbers to parts that had none: 5
