File: SMU V2/power.kicad_sch (KiCad schematic)
At the start: 7 parts

Commit message: v2 layout
Parts:
- removed TP301, TP303, TP304, TP305, TP306, TP307: SMD Test Point, bfr_utilities:TestPoint_Keystone_5019_Miniature, symbol bfr_utilities:SMD_Test_Point
- renumbered TP302 to TP301
Other:
- added sheet LDO (LDO.kicad_sch)
