File: SMU V2/vbatt_protection.kicad_sch (KiCad schematic)
At the start: 5 parts, among them Q1101 SI2301CDS-T1-GE3

Commit message: v2 layout
Parts:
- renumbered D1101 to D1201, F1101 to F1201, Q1101 to Q1201, R1101 to R1201, TVS1101 to TVS1201
Changed lines of the file:
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@@
 		(dnp no)
 		(fields_autoplaced yes)
-		(property "Reference" "F1101"
+		(property "Reference" "F1201"
 			(at 152.4 81.28 0)
 			(effects
@@
 			(project ""
 				(path "/1f58b889-96e6-4877-90a3-5a655db5910b/b9f10619-4e5b-45af-b866-c6815d605ed5/ffadd9c2-fe2d-4025-92ac-e8757544fe06"
-					(reference "F1101")
+					(reference "F1201")
 					(unit 1)
 				)
@@
 		(dnp no)
 		(fields_autoplaced yes)
-		(property "Reference" "#PWR01102"
+		(property "Reference" "#PWR01202"
 			(at 186.69 81.28 0)
 			(effects
@@
 			(project "SMU V1"
 				(path "/1f58b889-96e6-4877-90a3-5a655db5910b/b9f10619-4e5b-45af-b866-c6815d605ed5/ffadd9c2-fe2d-4025-92ac-e8757544fe06"
-					(reference "#PWR01102")
+					(reference "#PWR01202")
 					(unit 1)
 				)
@@
 		(on_board yes)
 		(dnp no)
-		(property "Reference" "TVS1101"
+		(property "Reference" "TVS1201"
 			(at 152.146 95.25 90)
 			(effects
@@
 			(project ""
 				(path "/1f58b889-96e6-4877-90a3-5a655db5910b/b9f10619-4e5b-45af-b866-c6815d605ed5/ffadd9c2-fe2d-4025-92ac-e8757544fe06"
-					(reference "TVS1101")
+					(reference "TVS1201")
 					(unit 1)
 				)
@@
 		(dnp no)
 		(fields_autoplaced yes)
-		(property "Reference" "D1101"
+		(property "Reference" "D1201"
 			(at 176.8475 63.5 0)
 			(effects
@@
 			(project ""
 				(path "/1f58b889-96e6-4877-90a3-5a655db5910b/b9f10619-4e5b-45af-b866-c6815d605ed5/ffadd9c2-fe2d-4025-92ac-e8757544fe06"
-					(reference "D1101")
+					(reference "D1201")
 					(unit 1)
 				)
@@
 		(dnp no)
 		(fields_autoplaced yes)
-		(property "Reference" "R1101"
+		(property "Reference" "R1201"
 			(at 167.64 64.77 0)
 			(effects
@@
 			(project ""
 				(path "/1f58b889-96e6-4877-90a3-5a655db5910b/b9f10619-4e5b-45af-b866-c6815d605ed5/ffadd9c2-fe2d-4025-92ac-e8757544fe06"
-					(reference "R1101")
+					(reference "R1201")
 					(unit 1)
 				)
@@
 		(dnp no)
 		(fields_autoplaced yes)
-		(property "Reference" "#PWR01101"
+		(property "Reference" "#PWR01201"
 			(at 133.35 119.38 0)
 			(effects
@@
 			(project ""
 				(path "/1f58b889-96e6-4877-90a3-5a655db5910b/b9f10619-4e5b-45af-b866-c6815d605ed5/ffadd9c2-fe2d-4025-92ac-e8757544fe06"
-					(reference "#PWR01101")
+					(reference "#PWR01201")
 					(unit 1)
 				)
@@
 		(on_board yes)
 		(dnp no)
-		(property "Reference" "Q1101"
+		(property "Reference" "Q1201"
 			(at 125.73 81.28 90)
 			(effects
@@
 			(project ""
 				(path "/1f58b889-96e6-4877-90a3-5a655db5910b/b9f10619-4e5b-45af-b866-c6815d605ed5/ffadd9c2-fe2d-4025-92ac-e8757544fe06"
-					(reference "Q1101")
+					(reference "Q1201")
 					(unit 1)
 				)
