File: SMU V3/Microcontroller.kicad_sch (KiCad schematic)
At the start: 5 parts

Commit message: improved V3
added uart/spi test points and status leds
removed main 3v3 ldo
added silkscreen
Parts:
- added D201: Green, Diode_SMD:D_0805_2012Metric_Pad1.15x1.40mm_HandSolder, symbol bfr_diodes:KT-0805G
- added D202: Yellow, Diode_SMD:D_0805_2012Metric_Pad1.15x1.40mm_HandSolder, symbol bfr_diodes:KT-0805Y
- added D203: Red, Diode_SMD:D_0603_1608Metric_Pad1.05x0.95mm_HandSolder, symbol bfr_diodes:KT-0603R
- added R201, R202, R203: 120, Resistor_SMD:R_0603_1608Metric_Pad0.98x0.95mm_HandSolder, symbol bfr_resistors:RMCF0603FT120R
- renumbered C1 to C201, C2 to C202, C3 to C203, C4 to C204, MCU1 to MCU201
Connections:
- net DISP_I2C_SCL: no longer MCU201.28 (PB13)
- net GND: now also D201.1 (K), D202.1 (K), D203.1 (K)
- net GPS_Error: now reaches MCU201.32 (PB12)
- net GPS_Error: now also R203.1
- net GPS_Standard: now reaches MCU201.36 (PB11)
- net GPS_Standard: now also R202.1
- net GPS_RTK: now reaches MCU201.40 (PB10)
- net GPS_RTK: now also R201.1
- new net: D201.2 (A), R201.2
- new net: D202.2 (A), R202.2
- new net: D203.2 (A), R203.2
- no-connect marks 13 -> 10
Other:
- note added: "GPS RTK working"
- note added: "GPS not working"
- note added: "GPS standard function working"
