File: SMU V3/gps.kicad_sch (KiCad schematic)
At the start: 8 parts

Commit message: improved V3
added uart/spi test points and status leds
removed main 3v3 ldo
added silkscreen
Parts:
- added TP501: GPS1_UART_RX, bfr_utilities:TestPoint_Keystone_5019_Miniature, symbol bfr_utilities:SMD_Test_Point
- added TP502: GPS1_UART_TX, bfr_utilities:TestPoint_Keystone_5019_Miniature, symbol bfr_utilities:SMD_Test_Point
- added TP503: GPS2_UART_RX, bfr_utilities:TestPoint_Keystone_5019_Miniature, symbol bfr_utilities:SMD_Test_Point
- added TP504: GPS2_UART_TX, bfr_utilities:TestPoint_Keystone_5019_Miniature, symbol bfr_utilities:SMD_Test_Point
- renumbered C9 to C501, C10 to C502, C11 to C503, C12 to C504, C13 to C505, C14 to C506, GPS1 to GPS501, GPS2 to GPS502
Connections:
- net GPS1.UART_RX: now also TP501.1
- net GPS1.UART_TX: now also TP502.1
- net GPS2.UART_RX: now also TP503.1
- net GPS2.UART_TX: now also TP504.1
Other:
- sheet GPS1 LDO ports: added GPS1_PGOOD; removed GPS_PGOOD
