File: SMU V3/imu.kicad_sch (KiCad schematic)
At the start: 3 parts, among them U1 LSM6DSOTR

Commit message: improved V3
added uart/spi test points and status leds
removed main 3v3 ldo
added silkscreen
Parts:
- added TP601: IMU_SPI_CS, bfr_utilities:TestPoint_Keystone_5019_Miniature, symbol bfr_utilities:SMD_Test_Point
- added TP602: IMU_SPI_MISO, bfr_utilities:TestPoint_Keystone_5019_Miniature, symbol bfr_utilities:SMD_Test_Point
- added TP603: IMU_SPI_MOSI, bfr_utilities:TestPoint_Keystone_5019_Miniature, symbol bfr_utilities:SMD_Test_Point
- added TP604: IMU_SPI_SCK, bfr_utilities:TestPoint_Keystone_5019_Miniature, symbol bfr_utilities:SMD_Test_Point
- renumbered C15 to C601, C16 to C602, U1 to U601
Connections:
- net IMU_SPI.CS: now also TP601.1
- net IMU_SPI.MISO: now also TP602.1
- net IMU_SPI.MOSI: now also TP603.1
- net IMU_SPI.SCK: now also TP604.1
