File: SMU V3/power.kicad_sch (KiCad schematic)
At the start: 1 part

Commit message: improved V3
added uart/spi test points and status leds
removed main 3v3 ldo
added silkscreen
Parts:
- renumbered TP1 to TP301
Other:
- removed sheet LDO
Changed lines of the file:
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@@
 		)
-	)
-	(junction
-		(at 190.5 81.28)
-		(diameter 0)
-		(color 0 0 0 0)
 	)
 	(wire
@@
 	(wire
 		(pts
-			(xy 190.5 81.28) (xy 190.5 105.41)
-		)
-		(stroke
-			(width 0)
-			(type default)
-		)
-	)
-	(wire
-		(pts
-			(xy 177.8 81.28) (xy 190.5 81.28)
-		)
-		(stroke
-			(width 0)
-			(type default)
-		)
-	)
-	(wire
-		(pts
-			(xy 190.5 105.41) (xy 196.85 105.41)
-		)
-		(stroke
-			(width 0)
-			(type default)
-		)
-	)
-	(wire
-		(pts
-			(xy 231.14 105.41) (xy 245.11 105.41)
-		)
-		(stroke
-			(width 0)
-			(type default)
-		)
-	)
-	(wire
-		(pts
-			(xy 190.5 81.28) (xy 215.9 81.28)
+			(xy 177.8 81.28) (xy 215.9 81.28)
 		)
 		(stroke
@@
 			)
 			(justify right)
-		)
-	)
-	(hierarchical_label "3V3"
-		(shape input)
-		(at 245.11 105.41 0)
-		(effects
-			(font
-				(size 1.27 1.27)
-			)
-			(justify left)
 		)
 	)
@@
 		(dnp no)
 		(fields_autoplaced yes)
-		(property "Reference" "#PWR06"
+		(property "Reference" "#PWR0301"
 			(at 73.66 133.35 0)
 			(hide yes)
@@
 			(project "SMU V3"
 				(path "/1f58b889-96e6-4877-90a3-5a655db5910b/b9f10619-4e5b-45af-b866-c6815d605ed5"
-					(reference "#PWR06")
+					(reference "#PWR0301")
 					(unit 1)
 				)
@@
 		(in_pos_files yes)
 		(dnp no)
-		(property "Reference" "TP1"
+		(property "Reference" "TP301"
 			(at 69.088 112.268 0)
 			(show_name no)
@@
 			(project "SMU V3"
 				(path "/1f58b889-96e6-4877-90a3-5a655db5910b/b9f10619-4e5b-45af-b866-c6815d605ed5"
-					(reference "TP1")
+					(reference "TP301")
 					(unit 1)
 				)
 			)
-		)
-	)
-	(sheet
-		(at 196.85 97.79)
-		(size 34.29 13.97)
-		(exclude_from_sim no)
-		(in_bom yes)
-		(on_board yes)
-		(dnp no)
-		(fields_autoplaced yes)
-		(stroke
-			(width 0.1524)
-			(type solid)
-		)
-		(fill
-			(color 255 255 194 1)
-		)
-		(property "Sheetname" "LDO"
-			(at 196.85 97.0784 0)
-			(show_name no)
-			(do_not_autoplace no)
-			(effects
-				(font
-					(size 1.27 1.27)
-				)
-				(justify left bottom)
-			)
-		)
-		(property "Sheetfile" "LDO.kicad_sch"
-			(at 196.85 112.3446 0)
-			(show_name no)
-			(do_not_autoplace no)
-			(effects
-				(font
-					(size 1.27 1.27)
-				)
-				(justify left top)
-			)
-		)
-		(pin "VIN" input
-			(at 196.85 105.41 180)
-			(effects
-				(font
-					(size 1.27 1.27)
-				)
-				(justify left)
-			)
-		)
-		(pin "VOUT" input
-			(at 231.14 105.41 0)
-			(effects
-				(font
-					(size 1.27 1.27)
-				)
-				(justify right)
-			)
-		)
-		(instances
-			(project "SMU V3"
-				(path "/1f58b889-96e6-4877-90a3-5a655db5910b/b9f10619-4e5b-45af-b866-c6815d605ed5"
-					(page "14")
-				)
-			)
